File: hw/adsr_vca_fx/SE8233X2_LDO.kicad_sch (KiCad schematic)
At the start: 6 parts, among them U10 SE8233X2

Commit message: first draft layout
Parts:
- renumbered C27 to C21, C28 to C22, R28 to R24, TP12 to TP9, U10 to U7
Changed lines of the file:
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@@
   (symbol (lib_id "Regulator_Linear:MCP1700x-330xxTT") (at 130.81 86.36 0) (unit 1)
     (in_bom yes) (on_board yes) (dnp no)
-    (property "Reference" "U10" (at 130.81 80.2132 0)
+    (property "Reference" "U7" (at 130.81 80.2132 0)
       (effects (font (size 1.27 1.27)))
     )
@@
       (project "adsr_vca_fx"
         (path "/2c7cc946-dcca-4ffb-b6a0-bf0c9ddb491b/d2509004-b5c4-4b3c-af62-d7c90bd19790/2b12c81b-590f-42b3-a93e-f9019ce43b66"
-          (reference "U10") (unit 1)
+          (reference "U7") (unit 1)
         )
       )
@@
   (symbol (lib_id "Device:C") (at 101.6 95.25 0) (unit 1)
     (in_bom yes) (on_board yes) (dnp no)
-    (property "Reference" "C27" (at 104.521 94.0816 0)
+    (property "Reference" "C21" (at 104.521 94.0816 0)
       (effects (font (size 1.27 1.27)) (justify left))
     )
@@
       (project "adsr_vca_fx"
         (path "/2c7cc946-dcca-4ffb-b6a0-bf0c9ddb491b/d2509004-b5c4-4b3c-af62-d7c90bd19790/2b12c81b-590f-42b3-a93e-f9019ce43b66"
-          (reference "C27") (unit 1)
+          (reference "C21") (unit 1)
         )
       )
@@
   (symbol (lib_id "Device:C") (at 161.29 95.25 0) (unit 1)
     (in_bom yes) (on_board yes) (dnp no)
-    (property "Reference" "C28" (at 164.211 94.0816 0)
+    (property "Reference" "C22" (at 164.211 94.0816 0)
       (effects (font (size 1.27 1.27)) (justify left))
     )
@@
       (project "adsr_vca_fx"
         (path "/2c7cc946-dcca-4ffb-b6a0-bf0c9ddb491b/d2509004-b5c4-4b3c-af62-d7c90bd19790/2b12c81b-590f-42b3-a93e-f9019ce43b66"
-          (reference "C28") (unit 1)
+          (reference "C22") (unit 1)
         )
       )
@@
   (symbol (lib_id "Device:R") (at 181.61 107.95 0) (unit 1)
     (in_bom yes) (on_board yes) (dnp no)
-    (property "Reference" "R28" (at 183.388 106.7816 0)
+    (property "Reference" "R24" (at 183.388 106.7816 0)
       (effects (font (size 1.27 1.27)) (justify left))
     )
@@
       (project "adsr_vca_fx"
         (path "/2c7cc946-dcca-4ffb-b6a0-bf0c9ddb491b/d2509004-b5c4-4b3c-af62-d7c90bd19790/2b12c81b-590f-42b3-a93e-f9019ce43b66"
-          (reference "R28") (unit 1)
+          (reference "R24") (unit 1)
         )
       )
@@
   (symbol (lib_id "Connector:TestPoint") (at 181.61 83.82 0) (unit 1)
     (in_bom yes) (on_board yes) (dnp no)
-    (property "Reference" "TP12" (at 183.0832 81.9912 0)
+    (property "Reference" "TP9" (at 183.0832 81.9912 0)
       (effects (font (size 1.27 1.27)) (justify left))
     )
@@
       (project "adsr_vca_fx"
         (path "/2c7cc946-dcca-4ffb-b6a0-bf0c9ddb491b/d2509004-b5c4-4b3c-af62-d7c90bd19790/2b12c81b-590f-42b3-a93e-f9019ce43b66"
-          (reference "TP12") (unit 1)
+          (reference "TP9") (unit 1)
         )
       )

Commit message: completed layout
Parts:
- removed TP9: TestPoint, TestPoint:TestPoint_Pad_D1.0mm, symbol Connector:TestPoint
Changed lines of the file:
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@@
-    (stroke (width 0) (type default))
-  )
-  (wire (pts (xy 181.61 86.36) (xy 181.61 83.82))
     (stroke (width 0) (type default))
   )
@@
         )
       )
-    )
-  )
-  (symbol (lib_id "Connector:TestPoint") (at 181.61 83.82 0) (unit 1)
-    (in_bom yes) (on_board yes) (dnp no)
-    (property "Reference" "TP9" (at 183.0832 81.9912 0)
-      (effects (font (size 1.27 1.27)) (justify left))
-    )
-    (property "Value" "TestPoint" (at 183.0832 83.1342 0)
-      (effects (font (size 1.27 1.27)) (justify left) hide)
-    )
-    (property "Footprint" "TestPoint:TestPoint_Pad_D1.0mm" (at 186.69 83.82 0)
-      (effects (font (size 1.27 1.27)) hide)
-    )
-    (property "Datasheet" "~" (at 186.69 83.82 0)
-      (effects (font (size 1.27 1.27)) hide)
-    )
-    (property "LcscNo" "~" (at 181.61 83.82 0)
-      (effects (font (size 1.27 1.27)) hide)
-    )
-    (property "Type" "~" (at 181.61 83.82 0)
-      (effects (font (size 1.27 1.27)) hide)
-    )
-    (pin "1")
-    (instances
-      (project "adsr_vca_fx"
-        (path "/2c7cc946-dcca-4ffb-b6a0-bf0c9ddb491b/d2509004-b5c4-4b3c-af62-d7c90bd19790/2b12c81b-590f-42b3-a93e-f9019ce43b66"
-          (reference "TP9") (unit 1)
-        )
-      )
