File: hw/adsr_vca_fx/_autosave-neg_pol_protection.kicad_sch (KiCad schematic)
At the start: 3 parts, among them Q1 HX2301A PMOS

Commit message: completed layout
Connections:
- net VIN: no longer Q1.3 (D)
- net VOUT: now also D1.2 (A); no longer D1.1 (K), Q1.2 (S)
- new net: D1.1 (K), R2.1
- now unconnected: Q1.1 (G)
Other:
- note removed: "See "MOSFET Protection" and fig3 for explanation of reverse polarity"
Changed lines of the file:
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@@
 (kicad_sch (version 20230121) (generator eeschema)
   (paper "A4")
-  (junction (at 128.27 102.87) (diameter 0) (color 0 0 0 0)
+  (junction (at 111.76 95.25) (diameter 0) (color 0 0 0 0)
   )
-  (junction (at 157.48 78.74) (diameter 0) (color 0 0 0 0)
+  (junction (at 140.97 71.12) (diameter 0) (color 0 0 0 0)
   )
-  (wire (pts (xy 128.27 102.87) (xy 128.27 110.49))
+  (wire (pts (xy 66.04 71.12) (xy 106.68 71.12))
     (stroke (width 0) (type default))
   )
-  (wire (pts (xy 157.48 95.25) (xy 157.48 102.87))
+  (wire (pts (xy 140.97 71.12) (xy 196.85 71.12))
     (stroke (width 0) (type default))
   )
-  (wire (pts (xy 128.27 118.11) (xy 128.27 127))
+  (wire (pts (xy 140.97 87.63) (xy 140.97 95.25))
     (stroke (width 0) (type default))
   )
-  (wire (pts (xy 157.48 87.63) (xy 157.48 78.74))
+  (wire (pts (xy 111.76 78.74) (xy 111.76 95.25))
     (stroke (width 0) (type default))
   )
-  (wire (pts (xy 82.55 78.74) (xy 123.19 78.74))
+  (wire (pts (xy 111.76 95.25) (xy 111.76 102.87))
     (stroke (width 0) (type default))
   )
-  (wire (pts (xy 157.48 78.74) (xy 213.36 78.74))
+  (wire (pts (xy 116.84 71.12) (xy 140.97 71.12))
     (stroke (width 0) (type default))
   )
-  (wire (pts (xy 128.27 86.36) (xy 128.27 102.87))
+  (wire (pts (xy 140.97 80.01) (xy 140.97 71.12))
     (stroke (width 0) (type default))
   )
-  (wire (pts (xy 133.35 78.74) (xy 157.48 78.74))
+  (wire (pts (xy 111.76 95.25) (xy 140.97 95.25))
     (stroke (width 0) (type default))
   )
-  (wire (pts (xy 128.27 102.87) (xy 157.48 102.87))
+  (wire (pts (xy 111.76 110.49) (xy 111.76 119.38))
     (stroke (width 0) (type default))
   )
-  (text "See \"MOSFET Protection\" and fig3 for explanation of reverse polarity"
-    (at 102.87 63.5 0)
-    (effects (font (size 1.27 1.27)) (justify left bottom) (href "https://sound-au.com/appnotes/an013.htm"))
-  )
-  (hierarchical_label "VOUT" (shape output) (at 213.36 78.74 0) (fields_autoplaced)
+  (hierarchical_label "VOUT" (shape output) (at 196.85 71.12 0) (fields_autoplaced)
     (effects (font (size 1.27 1.27)) (justify left))
   )
-  (hierarchical_label "VIN" (shape input) (at 82.55 78.74 180) (fields_autoplaced)
+  (hierarchical_label "VIN" (shape input) (at 66.04 71.12 180) (fields_autoplaced)
     (effects (font (size 1.27 1.27)) (justify right))
   )
-  (symbol (lib_id "Device:Q_PMOS_GSD") (at 128.27 81.28 90) (unit 1)
+  (symbol (lib_id "Device:Q_PMOS_GSD") (at 76.2 97.79 90) (unit 1)
     (in_bom yes) (on_board yes) (dnp no) (fields_autoplaced)
-    (property "Reference" "Q1" (at 128.27 72.39 90)
+    (property "Reference" "Q1" (at 76.2 88.9 90)
       (effects (font (size 1.27 1.27)))
     )
-    (property "Value" "HX2301A PMOS" (at 128.27 74.93 90)
+    (property "Value" "HX2301A PMOS" (at 76.2 91.44 90)
       (effects (font (size 1.27 1.27)))
     )
-    (property "Footprint" "Package_TO_SOT_SMD:SOT-23-3" (at 125.73 76.2 0)
+    (property "Footprint" "Package_TO_SOT_SMD:SOT-23-3" (at 73.66 92.71 0)
       (effects (font (size 1.27 1.27)) hide)
     )
-    (property "Datasheet" "${KIPRJMOD}/../../docs/datasheet/PMOS_HX2301A.pdf" (at 128.27 81.28 0)
+    (property "Datasheet" "${KIPRJMOD}/../../docs/datasheet/PMOS_HX2301A.pdf" (at 76.2 97.79 0)
       (effects (font (size 1.27 1.27)) hide)
     )
@@
           (reference "Q1") (unit 1)
         )
+        (path "/2c7cc946-dcca-4ffb-b6a0-bf0c9ddb491b/d2509004-b5c4-4b3c-af62-d7c90bd19790/3623950d-f622-45fd-aae1-ad3abdc5e2ad"
+          (reference "Q2") (unit 1)
+        )
       )
     )
   )
-  (symbol (lib_id "power:GND") (at 128.27 127 0) (unit 1)
+  (symbol (lib_id "Device:R") (at 111.76 106.68 0) (unit 1)
     (in_bom yes) (on_board yes) (dnp no) (fields_autoplaced)
-    (property "Reference" "#PWR011" (at 128.27 133.35 0)
+    (property "Reference" "R2" (at 114.3 106.045 0)
+      (effects (font (size 1.27 1.27)) (justify left))
+    )
+    (property "Value" "10K" (at 114.3 108.585 0)
+      (effects (font (size 1.27 1.27)) (justify left))
+    )
+    (property "Footprint" "Resistor_SMD:R_0805_2012Metric_Pad1.20x1.40mm_HandSolder" (at 109.982 106.68 90)
       (effects (font (size 1.27 1.27)) hide)
     )
-    (property "Value" "GND" (at 128.27 132.08 0)
+    (property "Datasheet" "~" (at 111.76 106.68 0)
+      (effects (font (size 1.27 1.27)) hide)
+    )
+    (pin "1")
+    (pin "2")
+    (instances
+      (project "adsr_vca_fx"
+        (path "/2c7cc946-dcca-4ffb-b6a0-bf0c9ddb491b/d2509004-b5c4-4b3c-af62-d7c90bd19790"
+          (reference "R2") (unit 1)
+        )
+        (path "/2c7cc946-dcca-4ffb-b6a0-bf0c9ddb491b/d2509004-b5c4-4b3c-af62-d7c90bd19790/7f56a6d0-e9ac-40b5-a9da-5532f531790a"
+          (reference "R25") (unit 1)
+        )
+        (path "/2c7cc946-dcca-4ffb-b6a0-bf0c9ddb491b/d2509004-b5c4-4b3c-af62-d7c90bd19790/3623950d-f622-45fd-aae1-ad3abdc5e2ad"
+          (reference "R26") (unit 1)
+        )
+      )
+    )
+  )
+  (symbol (lib_id "power:GND") (at 111.76 119.38 0) (unit 1)
+    (in_bom yes) (on_board yes) (dnp no) (fields_autoplaced)
+    (property "Reference" "#PWR011" (at 111.76 125.73 0)
+      (effects (font (size 1.27 1.27)) hide)
+    )
+    (property "Value" "GND" (at 111.76 124.46 0)
       (effects (font (size 1.27 1.27)))
     )
-    (property "Footprint" "" (at 128.27 127 0)
+    (property "Footprint" "" (at 111.76 119.38 0)
       (effects (font (size 1.27 1.27)) hide)
     )
-    (property "Datasheet" "" (at 128.27 127 0)
+    (property "Datasheet" "" (at 111.76 119.38 0)
       (effects (font (size 1.27 1.27)) hide)
     )
@@
           (reference "#PWR068") (unit 1)
         )
+        (path "/2c7cc946-dcca-4ffb-b6a0-bf0c9ddb491b/d2509004-b5c4-4b3c-af62-d7c90bd19790/3623950d-f622-45fd-aae1-ad3abdc5e2ad"
+          (reference "#PWR071") (unit 1)
+        )
       )
     )
   )
-  (symbol (lib_id "Device:D_Zener") (at 157.48 91.44 270) (unit 1)
+  (symbol (lib_id "Device:D_Zener") (at 140.97 83.82 90) (unit 1)
     (in_bom yes) (on_board yes) (dnp no) (fields_autoplaced)
-    (property "Reference" "D1" (at 160.02 90.805 90)
-      (effects (font (size 1.27 1.27)) (justify left))
+    (property "Reference" "D1" (at 143.51 83.185 90)
+      (effects (font (size 1.27 1.27)) (justify right))
     )
-    (property "Value" "BZT52C 12V" (at 160.02 93.345 90)
-      (effects (font (size 1.27 1.27)) (justify left))
+    (property "Value" "BZT52C 12V" (at 143.51 85.725 90)
+      (effects (font (size 1.27 1.27)) (justify right))
     )
-    (property "Footprint" "Diode_SMD:D_SOD-123F" (at 157.48 91.44 0)
+    (property "Footprint" "Diode_SMD:D_SOD-123F" (at 140.97 83.82 0)
       (effects (font (size 1.27 1.27)) hide)
     )
-    (property "Datasheet" "${KIPRJMOD}/../../docs/datasheet/BZT52_SER-1375261.pdf" (at 157.48 91.44 0)
+    (property "Datasheet" "${KIPRJMOD}/../../docs/datasheet/BZT52_SER-1375261.pdf" (at 140.97 83.82 0)
       (effects (font (size 1.27 1.27)) hide)
     )
@@
           (reference "D3") (unit 1)
         )
-      )
-    )
-  )
-  (symbol (lib_id "Device:R") (at 128.27 114.3 0) (unit 1)
-    (in_bom yes) (on_board yes) (dnp no) (fields_autoplaced)
-    (property "Reference" "R2" (at 130.81 113.665 0)
-      (effects (font (size 1.27 1.27)) (justify left))
-    )
-    (property "Value" "10K" (at 130.81 116.205 0)
-      (effects (font (size 1.27 1.27)) (justify left))
-    )
-    (property "Footprint" "Resistor_SMD:R_0805_2012Metric_Pad1.20x1.40mm_HandSolder" (at 126.492 114.3 90)
-      (effects (font (size 1.27 1.27)) hide)
-    )
-    (property "Datasheet" "~" (at 128.27 114.3 0)
-      (effects (font (size 1.27 1.27)) hide)
-    )
-    (pin "1")
-    (pin "2")
-    (instances
-      (project "adsr_vca_fx"
-        (path "/2c7cc946-dcca-4ffb-b6a0-bf0c9ddb491b/d2509004-b5c4-4b3c-af62-d7c90bd19790"
-          (reference "R2") (unit 1)
-        )
-        (path "/2c7cc946-dcca-4ffb-b6a0-bf0c9ddb491b/d2509004-b5c4-4b3c-af62-d7c90bd19790/7f56a6d0-e9ac-40b5-a9da-5532f531790a"
-          (reference "R25") (unit 1)
+        (path "/2c7cc946-dcca-4ffb-b6a0-bf0c9ddb491b/d2509004-b5c4-4b3c-af62-d7c90bd19790/3623950d-f622-45fd-aae1-ad3abdc5e2ad"
+          (reference "D4") (unit 1)
         )
       )
